File: IsolatorPanel.kicad_pcb (KiCad board)
At the start: 2 copper layers, 99.6 x 100 mm, 125 parts, among them J1 Step_0_In, J2 Step_0_Out, J3 Step_1_In, J4 Step_1_Out, J5 UART_In, J6 UART_Out, U1 ISO6741, U2 ISO6741, U3 ISO6721

Commit message: Switched RX and TX silkscreen
Other:
- board text added: "Power GND TX→ RX←"
- board text added: "Power GND →RX ←TX"
- board text removed: "Power GND RX← TX→"
- board text removed: "Power GND ←TX →RX"
Changed lines of the file:
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@@
   )
   (setup
-    (last_trace_width 0.254)
+    (last_trace_width 0.25)
     (user_trace_width 0.127)
     (user_trace_width 0.254)
@@
     (effects (font (size 2 2) (thickness 0.3)) (justify mirror))
   )
-  (gr_text "Power\nGND\n←TX\n→RX" (at 159.258 106.68) (layer B.SilkS)
+  (gr_text "Power\nGND\n→RX\n←TX" (at 159.258 106.68) (layer B.SilkS)
     (effects (font (size 1.5 1.5) (thickness 0.25)) (justify left mirror))
   )
@@
     (effects (font (size 1.5 1.5) (thickness 0.25)) (justify right mirror))
   )
-  (gr_text "Power\nGND\nRX←\nTX→" (at 134.493 106.68) (layer B.SilkS)
+  (gr_text "Power\nGND\nTX→\nRX←" (at 134.493 106.68) (layer B.SilkS)
     (effects (font (size 1.5 1.5) (thickness 0.25)) (justify right mirror))
   )
@@
     (effects (font (size 1 1) (thickness 0.15)))
   )
-  (gr_text "Power\nGND\nRX←\nTX→" (at 101.219 106.68) (layer B.SilkS)
+  (gr_text "Power\nGND\nTX→\nRX←" (at 101.219 106.68) (layer B.SilkS)
     (effects (font (size 1.5 1.5) (thickness 0.25)) (justify right mirror))
   )
@@
     (effects (font (size 2 2) (thickness 0.3)))
   )
-  (gr_text "Power\nGND\n←TX\n→RX" (at 125.984 106.68) (layer B.SilkS)
+  (gr_text "Power\nGND\n→RX\n←TX" (at 125.984 106.68) (layer B.SilkS)
     (effects (font (size 1.5 1.5) (thickness 0.25)) (justify left mirror))
   )
@@
     (effects (font (size 2 2) (thickness 0.3)) (justify mirror))
   )
-  (gr_text "Power\nGND\n←TX\n→RX" (at 92.71 106.68) (layer B.SilkS)
+  (gr_text "Power\nGND\n→RX\n←TX" (at 92.71 106.68) (layer B.SilkS)
     (effects (font (size 1.5 1.5) (thickness 0.25)) (justify left mirror))
   )
-  (gr_text "Power\nGND\nRX←\nTX→" (at 67.945 106.68) (layer B.SilkS)
+  (gr_text "Power\nGND\nTX→\nRX←" (at 67.945 106.68) (layer B.SilkS)
     (effects (font (size 1.5 1.5) (thickness 0.25)) (justify right mirror))
   )
